File: Schaltplan Steuerung/UV238.sch (KiCad schematic (older format))
At the start: 58 parts

Commit message: Schalttafel bis auf Abluftsteuerung fertig. Test steht aus.
Parts:
- gave numbers to parts that had none: 42
Connections:
- net Y32: no longer J22.1 (P1)
- net at K2.A1: now also K1.13; no longer K1.14
- net at S1.12, S3.13: now also K1.14; no longer K1.13
- net at S4.12, S6.13: now also K1.24; no longer K1.23
- net at K3.A1: now also K1.23; no longer K1.24
- net at S7.12, S9.13: now also K1.34; no longer K1.33
- net at K4.A1: now also K1.33; no longer K1.34
- new net Not-Halt_42: J22.1 (P1)
Other:
- note added: "Achtung! Dieser Taster ist durch das Relais\nK6 abgebildet, weil sonst zu wenige Leitungen\nim Steuerkabel vorhanden sind.\nKeine logische Invertierung!"
- note added: "K2.43"
- note added: "K2.44"
- moved on the sheet: K1B, K1C, K1D
